File: tiny_radio/tiny_radio.sch (KiCad schematic (older format))
At the start: 9 parts, among them IC1 ATTINY84-P, P1 CONN_4, P2 CONN_3X2, P3 CONN_2, U1 RFM12B

Commit message: moved block over
Connections:
- wire segments 56 -> 59
Other:
- moved on the sheet: C1, C2, P1, P2, R1, R2

Commit message: work in progress
Connections:
- net labels added: IRQ, MISO, MOSI, RADIO_SEL, RESET, SCL
Changed lines of the file:
@@
-EESchema Schematic File Version 2  date Mon 07 Jan 2013 21:19:53 GMT
-LIBS:power,/home/dave/Desktop/kicad/lib/rfm12b,/home/dave/Desktop/kicad/lib/atmel,device,transistors,conn,linear,regul,74xx,cmos4000,adc-dac,memory,xilinx,special,microcontrollers,dsp,microchip,analog_switches,motorola,texas,intel,audio,interface,digital-audio,philips,display,cypress,siliconi,opto,atmel,contrib,valves
+EESchema Schematic File Version 2  date Thu 10 Jan 2013 19:59:46 GMT
+LIBS:power
+LIBS:rfm12b
+LIBS:atmel
+LIBS:device
+LIBS:transistors
+LIBS:conn
+LIBS:linear
+LIBS:regul
+LIBS:74xx
+LIBS:cmos4000
+LIBS:adc-dac
+LIBS:memory
+LIBS:xilinx
+LIBS:special
+LIBS:microcontrollers
+LIBS:dsp
+LIBS:microchip
+LIBS:analog_switches
+LIBS:motorola
+LIBS:texas
+LIBS:intel
+LIBS:audio
+LIBS:interface
+LIBS:digital-audio
+LIBS:philips
+LIBS:display
+LIBS:cypress
+LIBS:siliconi
+LIBS:opto
+LIBS:contrib
+LIBS:valves
+LIBS:tiny_radio-cache
 EELAYER 24  0
 EELAYER END
 $Descr A4 11700 8267
+encoding utf-8
 Sheet 1 1
 Title "tiny radio"
-Date "6 jan 2013"
+Date "10 jan 2013"
 Rev "1"
 Comp ""
@@
 Comment4 ""
 $EndDescr
+Text Label 4100 5800 0    60   ~ 0
+RADIO_SEL
+Text Label 4100 5900 0    60   ~ 0
+IRQ
+Text Label 4100 6000 0    60   ~ 0
+RESET
+Text Label 4100 5400 0    60   ~ 0
+MOSI
+Text Label 4100 5300 0    60   ~ 0
+MISO
+Text Label 4100 5200 0    60   ~ 0
+SCL
 Wire Wire Line
 	5800 3950 5800 3850

Commit message: relayed and added rx/tx connector
Parts:
- removed P1: CONN_4, symbol CONN_4
- added P1: CONN_5, symbol CONN_5
Changed lines of the file:
@@
-EESchema Schematic File Version 2  date Thu 10 Jan 2013 19:59:46 GMT
+EESchema Schematic File Version 2  date Fri 25 Jan 2013 17:07:11 GMT
 LIBS:power
 LIBS:rfm12b
@@
 LIBS:valves
 LIBS:tiny_radio-cache
-EELAYER 24  0
+EELAYER 25  0
 EELAYER END
 $Descr A4 11700 8267
@@
 Sheet 1 1
 Title "tiny radio"
-Date "10 jan 2013"
+Date "25 jan 2013"
 Rev "1"
 Comp ""
@@
 Comment4 ""
 $EndDescr
+Wire Wire Line
+	4650 3700 4650 3750
+Connection ~ 6000 3850
+Wire Wire Line
+	6000 3850 5800 3850
+Wire Wire Line
+	5450 3500 5000 3500
+Connection ~ 5450 4700
+Wire Wire Line
+	5450 4400 5450 4700
+Wire Wire Line
+	4900 4550 4900 6000
+Wire Wire Line
+	4900 4550 5800 4550
+Wire Wire Line
+	5800 4550 5800 4450
+Connection ~ 6000 4800
+Wire Wire Line
+	6000 4450 6000 4800
+Wire Wire Line
+	4650 4050 4850 4050
+Wire Wire Line
+	4000 5500 4200 5500
+Connection ~ 7250 5700
+Wire Wire Line
+	7250 5700 7000 5700
+Wire Wire Line
+	7000 5700 7000 5800
+Wire Wire Line
+	6800 5600 6900 5600
+Connection ~ 6600 3800
+Wire Wire Line
+	4000 5800 4500 5800
+Wire Wire Line
+	4900 6000 4000 6000
+Wire Wire Line
+	1900 6000 1900 6100
+Wire Wire Line
+	5150 3700 5150 3600
+Wire Wire Line
+	5150 3600 5350 3600
+Wire Wire Line
+	5100 5700 5100 5850
+Wire Wire Line
+	6800 5200 7100 5200
+Wire Wire Line
+	7100 5200 7100 4700
+Wire Wire Line
+	7100 4700 4400 4700
+Wire Wire Line
+	4400 4700 4400 5200
+Wire Wire Line
+	6300 3900 6300 3800
+Wire Wire Line
+	6800 5100 7000 5100
+Wire Wire Line
+	7000 5100 7000 4800
+Wire Wire Line
+	7000 4800 4500 4800
+Wire Wire Line
+	4500 4800 4500 5800
+Wire Wire Line
+	5100 5100 4700 5100
+Wire Wire Line
+	6600 3900 6600 3700
+Wire Wire Line
+	6600 4300 6600 4500
+Wire Wire Line
+	6000 3800 6000 3950
+Wire Wire Line
+	4600 4900 4600 5300
+Wire Wire Line
+	4600 4900 6900 4900
+Wire Wire Line
+	6900 4900 6900 5300
+Wire Wire Line
+	6900 5300 6800 5300
+Wire Wire Line
+	4800 5200 4800 5900
+Wire Wire Line
+	4800 5200 5100 5200
+Wire Wire Line
+	6800 5700 6800 5800
+Wire Wire Line
+	5450 3500 5450 3600
+Wire Wire Line
+	5550 3600 5650 3600
+Wire Wire Line
+	5650 3600 5650 3650
+Wire Wire Line
+	1900 4700 1900 4800
+Wire Wire Line
+	4600 5300 4000 5300
+Wire Wire Line
+	4000 5400 4700 5400
+Wire Wire Line
+	4800 5900 4000 5900
+Wire Wire Line
+	4400 5200 4000 5200
+Wire Wire Line
+	6300 3800 6900 3800
+Wire Wire Line
+	6900 4300 6300 4300
+Connection ~ 6600 4300
+Wire Wire Line
+	6800 5500 7250 5500
+Wire Wire Line
+	7250 5500 7250 5900
+Wire Wire Line
+	4000 5100 4200 5100
+Wire Wire Line
+	4650 4300 4650 4150
+Wire Wire Line
+	4650 3950 4850 3950
+Connection ~ 5550 4550
+Wire Wire Line
+	5550 4400 5550 4550
+Wire Wire Line
+	5350 4400 5350 4900
+Connection ~ 5350 4900
+Wire Wire Line
+	5000 3500 5000 5100
+Connection ~ 5000 5100
+Wire Wire Line
+	4700 5400 4700 5100
+Wire Wire Line
+	5800 3850 5800 3950
+$Comp
+L CONN_5 P1
+U 1 1 5102A3FB
+P 4250 3950
+F 0 "P1" V 4200 3950 50  0000 C CNN
+F 1 "CONN_5" V 4300 3950 50  0000 C CNN
+	1    4250 3950
+	-1   0    0    1
+$EndComp
 Text Label 4100 5800 0    60   ~ 0
 RADIO_SEL
@@
 Text Label 4100 5200 0    60   ~ 0
 SCL
-Wire Wire Line
-	5800 3950 5800 3850
-Wire Wire Line
-	4700 5400 4700 5100
-Connection ~ 5000 5100
-Wire Wire Line
-	5000 5100 5000 3500
-Connection ~ 5350 4900
-Wire Wire Line
-	5350 4400 5350 4900
-Wire Wire Line
-	5550 4400 5550 4550
-Connection ~ 5550 4550
-Wire Wire Line
-	4650 3950 4850 3950
-Wire Wire Line
-	4650 4300 4650 4150
-Wire Wire Line
-	4000 5100 4200 5100
-Wire Wire Line
-	7250 5900 7250 5500
-Wire Wire Line
-	7250 5500 6800 5500
-Connection ~ 6600 4300
-Wire Wire Line
-	6900 4300 6300 4300
-Wire Wire Line
-	6900 3800 6300 3800
-Wire Wire Line
-	4000 5200 4400 5200
-Wire Wire Line
-	4000 5900 4800 5900
-Wire Wire Line
-	4700 5400 4000 5400
-Wire Wire Line
-	4000 5300 4600 5300
-Wire Wire Line
-	1900 4700 1900 4800
-Wire Wire Line
-	5650 3650 5650 3600
-Wire Wire Line
-	5650 3600 5550 3600
-Wire Wire Line
-	5450 3600 5450 3500
-Wire Wire Line
-	6800 5700 6800 5800
-Wire Wire Line
-	5100 5200 4800 5200
-Wire Wire Line
-	4800 5200 4800 5900
-Wire Wire Line
-	6800 5300 6900 5300
-Wire Wire Line
-	6900 5300 6900 4900
-Wire Wire Line
-	6900 4900 4600 4900
-Wire Wire Line
-	4600 4900 4600 5300
-Wire Wire Line
-	6000 3800 6000 3950
-Wire Wire Line
-	6600 4300 6600 4500
-Wire Wire Line
-	6600 3900 6600 3700
-Wire Wire Line
-	4700 5100 5100 5100
-Wire Wire Line
-	4500 4800 4500 5800
-Wire Wire Line
-	4500 4800 7000 4800
-Wire Wire Line
-	7000 4800 7000 5100
-Wire Wire Line
-	7000 5100 6800 5100
-Wire Wire Line
-	6300 3800 6300 3900
-Wire Wire Line
-	4400 5200 4400 4700
-Wire Wire Line
-	4400 4700 7100 4700
-Wire Wire Line
-	7100 4700 7100 5200
-Wire Wire Line
-	7100 5200 6800 5200
-Wire Wire Line
-	5100 5700 5100 5850
-Wire Wire Line
-	5350 3600 5150 3600
-Wire Wire Line
-	5150 3600 5150 3700
-Wire Wire Line
-	1900 6000 1900 6100
-Wire Wire Line
-	4000 6000 4900 6000
-Wire Wire Line
-	4500 5800 4000 5800
-Connection ~ 6600 3800
-Wire Wire Line
-	6800 5600 6900 5600
-Wire Wire Line
-	7000 5800 7000 5700
-Wire Wire Line
-	7000 5700 7250 5700
-Connection ~ 7250 5700
-Wire Wire Line
-	4000 5500 4200 5500
-Wire Wire Line
-	4650 3700 4650 3850
-Wire Wire Line
-	4650 4050 4850 4050
-Wire Wire Line
-	6000 4450 6000 4800
-Connection ~ 6000 4800
-Wire Wire Line
-	5800 4450 5800 4550
-Wire Wire Line
-	5800 4550 4900 4550
-Wire Wire Line
-	4900 4550 4900 6000
-Wire Wire Line
-	5450 4400 5450 4700
-Connection ~ 5450 4700
-Wire Wire Line
-	5450 3500 5000 3500
-Wire Wire Line
-	5800 3850 6000 3850
-Connection ~ 6000 3850
 Text Label 4750 4050 0    60   ~ 0
 Rx
@@
 Tx
 $Comp
-L +3.3V #PWR01
+L +3.3V #PWR3
 U 1 1 50E9A7B9
 P 4650 3700
-F 0 "#PWR01" H 4650 3660 30  0001 C CNN
+F 0 "#PWR3" H 4650 3660 30  0001 C CNN
 F 1 "+3.3V" H 4650 3810 30  0000 C CNN
 	1    4650 3700
@@
 $EndComp
 $Comp
-L GND #PWR02
+L GND #PWR4
 U 1 1 50E9A7B3
 P 4650 4300
-F 0 "#PWR02" H 4650 4300 30  0001 C CNN
+F 0 "#PWR4" H 4650 4300 30  0001 C CNN
 F 1 "GND" H 4650 4230 30  0001 C CNN
 	1    4650 4300
@@
 Text Label 4100 5100 0    60   ~ 0
 Tx
-$Comp
-L CONN_4 P1
-U 1 1 50E9A727
-P 4300 4000
-F 0 "P1" V 4250 4000 50  0000 C CNN
-F 1 "CONN_4" V 4350 4000 50  0000 C CNN
-	1    4300 4000
-	-1   0    0    1
-$EndComp
 $Comp
 L CONN_2 P3
@@
 $EndComp
 $Comp
-L GND #PWR03
+L GND #PWR2
 U 1 1 50E9905C
 P 1900 6100
-F 0 "#PWR03" H 1900 6100 30  0001 C CNN
+F 0 "#PWR2" H 1900 6100 30  0001 C CNN
 F 1 "GND" H 1900 6030 30  0001 C CNN
 	1    1900 6100
@@
 $EndComp
 $Comp
-L +3.3V #PWR04
+L +3.3V #PWR1
 U 1 1 50E99057
 P 1900 4700
-F 0 "#PWR04" H 1900 4660 30  0001 C CNN
+F 0 "#PWR1" H 1900 4660 30  0001 C CNN
 F 1 "+3.3V" H 1900 4810 30  0000 C CNN
 	1    1900 4700
@@
 $EndComp
 $Comp
-L GND #PWR05
+L GND #PWR7
 U 1 1 50E98FD6
 P 5650 3650
-F 0 "#PWR05" H 5650 3650 30  0001 C CNN
+F 0 "#PWR7" H 5650 3650 30  0001 C CNN
 F 1 "GND" H 5650 3580 30  0001 C CNN
 	1    5650 3650
@@
 $EndComp
 $Comp
-L +3.3V #PWR06
+L +3.3V #PWR6
 U 1 1 50E98FC4
 P 5150 3700
-F 0 "#PWR06" H 5150 3660 30  0001 C CNN
+F 0 "#PWR6" H 5150 3660 30  0001 C CNN
 F 1 "+3.3V" H 5150 3810 30  0000 C CNN
 	1    5150 3700
@@
 $EndComp
 $Comp
-L +3.3V #PWR07
+L +3.3V #PWR11
 U 1 1 50E98E7C
 P 6900 5600
-F 0 "#PWR07" H 6900 5560 30  0001 C CNN
+F 0 "#PWR11" H 6900 5560 30  0001 C CNN
 F 1 "+3.3V" H 6900 5710 30  0000 C CNN
 	1    6900 5600
@@
 $EndComp
 $Comp
-L GND #PWR08
+L GND #PWR12
 U 1 1 50E98E6A
 P 7250 5900
-F 0 "#PWR08" H 7250 5900 30  0001 C CNN
+F 0 "#PWR12" H 7250 5900 30  0001 C CNN
 F 1 "GND" H 7250 5830 30  0001 C CNN
 	1    7250 5900
@@
 $EndComp
 $Comp
-L GND #PWR09
+L GND #PWR5
 U 1 1 50E98E5E
 P 5100 5850
-F 0 "#PWR09" H 5100 5850 30  0001 C CNN
+F 0 "#PWR5" H 5100 5850 30  0001 C CNN
 F 1 "GND" H 5100 5780 30  0001 C CNN
 	1    5100 5850
@@
 $EndComp
 $Comp
-L +3.3V #PWR010
+L +3.3V #PWR8
 U 1 1 50E952D1
 P 6000 3800
-F 0 "#PWR010" H 6000 3760 30  0001 C CNN
+F 0 "#PWR8" H 6000 3760 30  0001 C CNN
 F 1 "+3.3V" H 6000 3910 30  0000 C CNN
 	1    6000 3800
@@
 $EndComp
 $Comp
-L GND #PWR011
+L GND #PWR10
 U 1 1 50E9522C
 P 6600 4500
-F 0 "#PWR011" H 6600 4500 30  0001 C CNN
+F 0 "#PWR10" H 6600 4500 30  0001 C CNN
 F 1 "GND" H 6600 4430 30  0001 C CNN
 	1    6600 4500
@@
 $EndComp
 $Comp
-L +3.3V #PWR012
+L +3.3V #PWR9
 U 1 1 50E95223
 P 6600 3700
-F 0 "#PWR012" H 6600 3660 30  0001 C CNN
+F 0 "#PWR9" H 6600 3660 30  0001 C CNN
 F 1 "+3.3V" H 6600 3810 30  0000 C CNN
 	1    6600 3700
@@
 $EndComp
 $Comp
-L PWR_FLAG #FLG013
+L PWR_FLAG #FLG2
 U 1 1 50E95196
 P 6900 4300
-F 0 "#FLG013" H 6900 4570 30  0001 C CNN
+F 0 "#FLG2" H 6900 4570 30  0001 C CNN
 F 1 "PWR_FLAG" H 6900 4530 30  0000 C CNN
 	1    6900 4300
@@
 $EndComp
 $Comp
-L PWR_FLAG #FLG014
+L PWR_FLAG #FLG1
 U 1 1 50E950A5
 P 6900 3800
-F 0 "#FLG014" H 6900 4070 30  0001 C CNN
+F 0 "#FLG1" H 6900 4070 30  0001 C CNN
 F 1 "PWR_FLAG" H 6900 4030 30  0000 C CNN
 	1    6900 3800
