File: optical_mouse/optical_mouse.sch (KiCad schematic (older format))
At the start: 12 parts

Commit message: first stab at circuit
Parts:
- added ???: ANDS-2610, symbol ANDS-2610
- added C?: CP1, ~, symbol CP1
Connections:
- wire segments 18 -> 40
Other:
- moved on the sheet: C?, X?
Changed lines of the file:
@@
 LIBS:contrib
 LIBS:valves
-LIBS:arduino
+LIBS:adns-2610
+LIBS:optical_mouse-cache
 EELAYER 27 0
 EELAYER END
@@
 L C C?
 U 1 1 5568675B
-P 5950 4400
-F 0 "C?" H 5950 4500 40  0000 L CNN
-F 1 "C" H 5956 4315 40  0000 L CNN
-F 2 "~" H 5988 4250 30  0000 C CNN
-F 3 "~" H 5950 4400 60  0000 C CNN
-	1    5950 4400
+P 5850 1850
+F 0 "C?" H 5850 1950 40  0000 L CNN
+F 1 "C" H 5856 1765 40  0000 L CNN
+F 2 "~" H 5888 1700 30  0000 C CNN
+F 3 "~" H 5850 1850 60  0000 C CNN
+	1    5850 1850
 	1    0    0    -1
 $EndComp
@@
 L CP1 C?
 U 1 1 5568676A
-P 6450 4400
-F 0 "C?" H 6500 4500 50  0000 L CNN
-F 1 "CP1" H 6500 4300 50  0000 L CNN
-F 2 "~" H 6450 4400 60  0000 C CNN
-F 3 "~" H 6450 4400 60  0000 C CNN
-	1    6450 4400
+P 6150 1850
+F 0 "C?" H 6200 1950 50  0000 L CNN
+F 1 "CP1" H 6200 1750 50  0000 L CNN
+F 2 "~" H 6150 1850 60  0000 C CNN
+F 3 "~" H 6150 1850 60  0000 C CNN
+	1    6150 1850
 	1    0    0    -1
 $EndComp
@@
 L CRYSTAL X?
 U 1 1 556867CB
-P 5950 5000
-F 0 "X?" H 5950 5150 60  0000 C CNN
-F 1 "CRYSTAL" H 5950 4850 60  0000 C CNN
-F 2 "~" H 5950 5000 60  0000 C CNN
-F 3 "~" H 5950 5000 60  0000 C CNN
-	1    5950 5000
-	1    0    0    -1
+P 8250 3000
+F 0 "X?" H 8250 3150 60  0000 C CNN
+F 1 "CRYSTAL" H 8250 2850 60  0000 C CNN
+F 2 "~" H 8250 3000 60  0000 C CNN
+F 3 "~" H 8250 3000 60  0000 C CNN
+	1    8250 3000
+	0    -1   -1   0
 $EndComp
 $Comp
@@
 Wire Wire Line
 	4700 3450 4700 2200
+$Comp
+L ANDS-2610 ???
+U 1 1 55686C9F
+P 6350 3250
+F 0 "???" H 6350 3250 60  0000 C CNN
+F 1 "ANDS-2610" H 6350 3250 60  0000 C CNN
+F 2 "" H 6350 3250 60  0000 C CNN
+F 3 "" H 6350 3250 60  0000 C CNN
+	1    6350 3250
+	1    0    0    -1
+$EndComp
+$Comp
+L +5V #PWR?
+U 1 1 55686CCD
+P 6450 1250
+F 0 "#PWR?" H 6450 1340 20  0001 C CNN
+F 1 "+5V" H 6450 1340 30  0000 C CNN
+F 2 "" H 6450 1250 60  0000 C CNN
+F 3 "" H 6450 1250 60  0000 C CNN
+	1    6450 1250
+	1    0    0    -1
+$EndComp
+Wire Wire Line
+	8250 2700 7550 2700
+Wire Wire Line
+	7550 2700 7550 2850
+Wire Wire Line
+	7550 3250 8000 3250
+Wire Wire Line
+	8000 3250 8000 3300
+Wire Wire Line
+	8000 3300 8250 3300
+Wire Wire Line
+	6450 1250 6450 2050
+Wire Wire Line
+	6450 1450 5850 1450
+Wire Wire Line
+	5850 1450 5850 1650
+Connection ~ 6450 1450
+Wire Wire Line
+	6150 1450 6150 1650
+Connection ~ 6150 1450
+$Comp
+L GND #PWR?
+U 1 1 55686E81
+P 5850 2900
+F 0 "#PWR?" H 5850 2900 30  0001 C CNN
+F 1 "GND" H 5850 2830 30  0001 C CNN
+F 2 "" H 5850 2900 60  0000 C CNN
+F 3 "" H 5850 2900 60  0000 C CNN
+	1    5850 2900
+	1    0    0    -1
+$EndComp
+Wire Wire Line
+	5850 2900 5850 2050
+Wire Wire Line
+	5950 2750 5850 2750
+Connection ~ 5850 2750
+Wire Wire Line
+	6150 2050 6150 2150
+Wire Wire Line
+	6150 2150 5850 2150
+Connection ~ 5850 2150
+$Comp
+L CP1 C?
+U 1 1 55686FA6
+P 7850 4050
+F 0 "C?" H 7900 4150 50  0000 L CNN
+F 1 "CP1" H 7900 3950 50  0000 L CNN
+F 2 "~" H 7850 4050 60  0000 C CNN
+F 3 "~" H 7850 4050 60  0000 C CNN
+	1    7850 4050
+	1    0    0    -1
+$EndComp
+Wire Wire Line
+	7550 3650 7850 3650
+Wire Wire Line
+	7850 3650 7850 3850
+$Comp
+L GND #PWR?
+U 1 1 55686FDA
+P 7850 4450
+F 0 "#PWR?" H 7850 4450 30  0001 C CNN
+F 1 "GND" H 7850 4380 30  0001 C CNN
+F 2 "" H 7850 4450 60  0000 C CNN
+F 3 "" H 7850 4450 60  0000 C CNN
+	1    7850 4450
+	1    0    0    -1
+$EndComp
+Wire Wire Line
+	7850 4450 7850 4250
+Wire Wire Line
+	4300 2500 5500 2500
+Wire Wire Line
+	5500 2500 5500 3550
+Wire Wire Line
+	5500 3550 5950 3550
+Wire Wire Line
+	4300 2600 5650 2600
+Wire Wire Line
+	5650 2600 5650 3150
+Wire Wire Line
+	5650 3150 5950 3150
 $EndSCHEMATC

Commit message: wip
Parts:
- gave numbers to parts that had none: 14
Connections:
- wire segments 40 -> 41
- no-connect marks 0 -> 22
Other:
- moved on the sheet: ??1, C1, C2, C3, D1, D2, D3, D4, R1, R2, R3, R4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
