File: optical_mouse/optical_mouse.sch (KiCad schematic (older format))
At the start: 14 parts, among them U1 ARDUINO_MINI, X1 CRYSTAL

Commit message: wip
Parts:
- removed X1: CRYSTAL, ~, symbol CRYSTAL
- added Y?: RESONATEUR, symbol RESONATEUR
Connections:
- wire segments 41 -> 43
Other:
- moved on the sheet: D1, D2, D3, D4, R1, R2, R3, R4
Changed lines of the file:
@@
 LIBS:valves
 LIBS:adns-2610
+LIBS:Resonator_3pins
+LIBS:arduino
 LIBS:optical_mouse-cache
 EELAYER 27 0
@@
 L LED D1
 U 1 1 55686723
-P 4200 2500
-F 0 "D1" H 4200 2600 50  0000 C CNN
-F 1 "LED" H 4200 2400 50  0000 C CNN
-F 2 "~" H 4200 2500 60  0000 C CNN
-F 3 "~" H 4200 2500 60  0000 C CNN
-	1    4200 2500
+P 4200 3100
+F 0 "D1" H 4200 3200 50  0000 C CNN
+F 1 "LED" H 4200 3000 50  0000 C CNN
+F 2 "~" H 4200 3100 60  0000 C CNN
+F 3 "~" H 4200 3100 60  0000 C CNN
+	1    4200 3100
 	0    1    1    0
 $EndComp
@@
 L R R1
 U 1 1 5568674C
-P 4200 3050
-F 0 "R1" V 4280 3050 40  0000 C CNN
-F 1 "R" V 4207 3051 40  0000 C CNN
-F 2 "~" V 4130 3050 30  0000 C CNN
-F 3 "~" H 4200 3050 30  0000 C CNN
-	1    4200 3050
+P 4200 2550
+F 0 "R1" V 4280 2550 40  0000 C CNN
+F 1 "R" V 4207 2551 40  0000 C CNN
+F 2 "~" V 4130 2550 30  0000 C CNN
+F 3 "~" H 4200 2550 30  0000 C CNN
+	1    4200 2550
 	1    0    0    -1
 $EndComp
@@
 $EndComp
 $Comp
-L CRYSTAL X1
-U 1 1 556867CB
-P 7750 4100
-F 0 "X1" H 7750 4250 60  0000 C CNN
-F 1 "CRYSTAL" H 7750 3950 60  0000 C CNN
-F 2 "~" H 7750 4100 60  0000 C CNN
-F 3 "~" H 7750 4100 60  0000 C CNN
-	1    7750 4100
-	0    -1   -1   0
-$EndComp
-$Comp
 L +5V #PWR01
 U 1 1 55686809
@@
 Wire Wire Line
 	3100 6000 3100 5800
-Wire Wire Line
-	4200 2700 4200 2800
-$Comp
-L +5V #PWR03
-U 1 1 556868DA
-P 4200 2150
-F 0 "#PWR03" H 4200 2240 20  0001 C CNN
-F 1 "+5V" H 4200 2240 30  0000 C CNN
-F 2 "" H 4200 2150 60  0000 C CNN
-F 3 "" H 4200 2150 60  0000 C CNN
-	1    4200 2150
-	1    0    0    -1
-$EndComp
 $Comp
 L LED D2
 U 1 1 556868F7
-P 4400 2500
-F 0 "D2" H 4400 2600 50  0000 C CNN
-F 1 "LED" H 4400 2400 50  0000 C CNN
-F 2 "~" H 4400 2500 60  0000 C CNN
-F 3 "~" H 4400 2500 60  0000 C CNN
-	1    4400 2500
+P 4400 3100
+F 0 "D2" H 4400 3200 50  0000 C CNN
+F 1 "LED" H 4400 3000 50  0000 C CNN
+F 2 "~" H 4400 3100 60  0000 C CNN
+F 3 "~" H 4400 3100 60  0000 C CNN
+	1    4400 3100
 	0    1    1    0
 $EndComp
@@
 L R R2
 U 1 1 556868FD
-P 4400 3050
-F 0 "R2" V 4480 3050 40  0000 C CNN
-F 1 "R" V 4407 3051 40  0000 C CNN
-F 2 "~" V 4330 3050 30  0000 C CNN
-F 3 "~" H 4400 3050 30  0000 C CNN
-	1    4400 3050
-	1    0    0    -1
-$EndComp
-Wire Wire Line
-	4400 2700 4400 2800
+P 4400 2550
+F 0 "R2" V 4480 2550 40  0000 C CNN
+F 1 "R" V 4407 2551 40  0000 C CNN
+F 2 "~" V 4330 2550 30  0000 C CNN
+F 3 "~" H 4400 2550 30  0000 C CNN
+	1    4400 2550
+	1    0    0    -1
+$EndComp
 $Comp
 L LED D3
 U 1 1 5568690C
-P 4600 2500
-F 0 "D3" H 4600 2600 50  0000 C CNN
-F 1 "LED" H 4600 2400 50  0000 C CNN
-F 2 "~" H 4600 2500 60  0000 C CNN
-F 3 "~" H 4600 2500 60  0000 C CNN
-	1    4600 2500
+P 4600 3100
+F 0 "D3" H 4600 3200 50  0000 C CNN
+F 1 "LED" H 4600 3000 50  0000 C CNN
+F 2 "~" H 4600 3100 60  0000 C CNN
+F 3 "~" H 4600 3100 60  0000 C CNN
+	1    4600 3100
 	0    1    1    0
 $EndComp
@@
 L R R3
 U 1 1 55686912
-P 4600 3050
-F 0 "R3" V 4680 3050 40  0000 C CNN
-F 1 "R" V 4607 3051 40  0000 C CNN
-F 2 "~" V 4530 3050 30  0000 C CNN
-F 3 "~" H 4600 3050 30  0000 C CNN
-	1    4600 3050
-	1    0    0    -1
-$EndComp
-Wire Wire Line
-	4600 2700 4600 2800
+P 4600 2550
+F 0 "R3" V 4680 2550 40  0000 C CNN
+F 1 "R" V 4607 2551 40  0000 C CNN
+F 2 "~" V 4530 2550 30  0000 C CNN
+F 3 "~" H 4600 2550 30  0000 C CNN
+	1    4600 2550
+	1    0    0    -1
+$EndComp
 $Comp
 L LED D4
 U 1 1 55686920
-P 4800 2500
-F 0 "D4" H 4800 2600 50  0000 C CNN
-F 1 "LED" H 4800 2400 50  0000 C CNN
-F 2 "~" H 4800 2500 60  0000 C CNN
-F 3 "~" H 4800 2500 60  0000 C CNN
-	1    4800 2500
+P 4800 3100
+F 0 "D4" H 4800 3200 50  0000 C CNN
+F 1 "LED" H 4800 3000 50  0000 C CNN
+F 2 "~" H 4800 3100 60  0000 C CNN
+F 3 "~" H 4800 3100 60  0000 C CNN
+	1    4800 3100
 	0    1    1    0
 $EndComp
@@
 L R R4
 U 1 1 55686926
-P 4800 3050
-F 0 "R4" V 4880 3050 40  0000 C CNN
-F 1 "R" V 4807 3051 40  0000 C CNN
-F 2 "~" V 4730 3050 30  0000 C CNN
-F 3 "~" H 4800 3050 30  0000 C CNN
-	1    4800 3050
-	1    0    0    -1
-$EndComp
-Wire Wire Line
-	4800 2700 4800 2800
+P 4800 2550
+F 0 "R4" V 4880 2550 40  0000 C CNN
+F 1 "R" V 4807 2551 40  0000 C CNN
+F 2 "~" V 4730 2550 30  0000 C CNN
+F 3 "~" H 4800 2550 30  0000 C CNN
+	1    4800 2550
+	1    0    0    -1
+$EndComp
 Wire Wire Line
 	3800 4850 4800 4850
 Wire Wire Line
-	4800 4850 4800 3300
-Wire Wire Line
 	3800 4750 4600 4750
 Wire Wire Line
-	4600 4750 4600 3300
-Wire Wire Line
 	3800 4650 4400 4650
 Wire Wire Line
-	4400 4650 4400 3300
-Wire Wire Line
 	3800 4550 4200 4550
-Wire Wire Line
-	4200 4550 4200 3300
 $Comp
 L ANDS-2610 ??1
@@
 $EndComp
 Wire Wire Line
-	7750 3800 7050 3800
-Wire Wire Line
-	7050 3800 7050 3950
-Wire Wire Line
-	7050 4350 7500 4350
-Wire Wire Line
-	7500 4350 7500 4400
-Wire Wire Line
-	7500 4400 7750 4400
-Wire Wire Line
 	5950 2350 5950 3150
 Wire Wire Line
@@
 Wire Wire Line
 	5000 4650 5450 4650
-Wire Wire Line
-	4200 2150 4200 2300
-Wire Wire Line
-	4200 2200 4800 2200
-Wire Wire Line
-	4400 2200 4400 2300
-Connection ~ 4200 2200
-Wire Wire Line
-	4800 2200 4800 2300
-Connection ~ 4400 2200
-Wire Wire Line
-	4600 2300 4600 2200
-Connection ~ 4600 2200
 NoConn ~ 3250 3100
 NoConn ~ 2950 3100
@@
 Wire Wire Line
 	5150 3800 3800 3800
+Wire Wire Line
+	4200 2800 4200 2900
+Wire Wire Line
+	4400 2800 4400 2900
+Wire Wire Line
+	4600 2800 4600 2900
+Wire Wire Line
+	4800 2800 4800 2900
+Wire Wire Line
+	4200 4550 4200 3300
+Wire Wire Line
+	4400 4650 4400 3300
+Wire Wire Line
+	4600 4750 4600 3300
+Wire Wire Line
+	4800 4850 4800 3300
+$Comp
+L +5V #PWR?
+U 1 1 556894CB
+P 4500 2100
+F 0 "#PWR?" H 4500 2190 20  0001 C CNN
+F 1 "+5V" H 4500 2190 30  0000 C CNN
+F 2 "" H 4500 2100 60  0000 C CNN
+F 3 "" H 4500 2100 60  0000 C CNN
+	1    4500 2100
+	1    0    0    -1
+$EndComp
+Wire Wire Line
+	4200 2300 4200 2200
+Wire Wire Line
+	4200 2200 4800 2200
+Wire Wire Line
+	4800 2200 4800 2300
+Wire Wire Line
+	4500 2100 4500 2200
+Connection ~ 4500 2200
+Wire Wire Line
+	4400 2300 4400 2200
+Connection ~ 4400 2200
+Wire Wire Line
+	4600 2300 4600 2200
+Connection ~ 4600 2200
+$Comp
+L RESONATEUR Y?
+U 1 1 55689636
+P 7800 4150
+F 0 "Y?" H 7820 4350 60  0000 C CNN
+F 1 "RESONATEUR" H 8230 3950 60  0000 C CNN
+F 2 "" H 7800 4150 60  0000 C CNN
+F 3 "" H 7800 4150 60  0000 C CNN
+	1    7800 4150
+	0    -1   -1   0
+$EndComp
+Wire Wire Line
+	7050 3950 7300 3950
+Wire Wire Line
+	7300 3950 7300 3850
+Wire Wire Line
+	7300 3850 7750 3850
+Wire Wire Line
+	7050 4350 7300 4350
+Wire Wire Line
+	7300 4350 7300 4450
+Wire Wire Line
+	7300 4450 7750 4450
 $EndSCHEMATC

Commit message: first viable layout
Parts:
- removed Y?: RESONATEUR, symbol RESONATEUR
- added Q1: CSTLS_G, murata-resonators-CSTLS_G8, symbol CSTLS_G
Connections:
- wire segments 43 -> 47
Other:
- moved on the sheet: ??1, C1, C2, C3
Changed lines of the file:
@@
 LIBS:Resonator_3pins
 LIBS:arduino
+LIBS:murata-resonators
 LIBS:optical_mouse-cache
 EELAYER 27 0
@@
 Sheet 1 1
 Title "Optical Mouse Camera"
-Date "29 may 2015"
+Date "31 may 2015"
 Rev ""
 Comp ""
@@
 L C C1
 U 1 1 5568675B
-P 5350 2950
-F 0 "C1" H 5350 3050 40  0000 L CNN
-F 1 "C" H 5356 2865 40  0000 L CNN
-F 2 "~" H 5388 2800 30  0000 C CNN
-F 3 "~" H 5350 2950 60  0000 C CNN
-	1    5350 2950
+P 5350 2900
+F 0 "C1" H 5350 3000 40  0000 L CNN
+F 1 "C" H 5356 2815 40  0000 L CNN
+F 2 "~" H 5388 2750 30  0000 C CNN
+F 3 "~" H 5350 2900 60  0000 C CNN
+	1    5350 2900
 	1    0    0    -1
 $EndComp
@@
 L CP1 C2
 U 1 1 5568676A
-P 5650 2950
-F 0 "C2" H 5700 3050 50  0000 L CNN
-F 1 "CP1" H 5700 2850 50  0000 L CNN
-F 2 "~" H 5650 2950 60  0000 C CNN
-F 3 "~" H 5650 2950 60  0000 C CNN
-	1    5650 2950
+P 5650 2900
+F 0 "C2" H 5700 3000 50  0000 L CNN
+F 1 "CP1" H 5700 2800 50  0000 L CNN
+F 2 "~" H 5650 2900 60  0000 C CNN
+F 3 "~" H 5650 2900 60  0000 C CNN
+	1    5650 2900
 	1    0    0    -1
 $EndComp
@@
 	1    0    0    -1
 $EndComp
-Wire Wire Line
-	3800 4850 4800 4850
-Wire Wire Line
-	3800 4750 4600 4750
-Wire Wire Line
-	3800 4650 4400 4650
-Wire Wire Line
-	3800 4550 4200 4550
 $Comp
 L ANDS-2610 ??1
 U 1 1 55686C9F
-P 5850 4350
-F 0 "??1" H 5850 4350 60  0000 C CNN
-F 1 "ANDS-2610" H 5850 4350 60  0000 C CNN
-F 2 "" H 5850 4350 60  0000 C CNN
-F 3 "" H 5850 4350 60  0000 C CNN
-	1    5850 4350
-	1    0    0    -1
-$EndComp
-$Comp
-L +5V #PWR04
+P 5850 4300
+F 0 "??1" H 5850 4300 60  0000 C CNN
+F 1 "ANDS-2610" H 5850 4300 60  0000 C CNN
+F 2 "" H 5850 4300 60  0000 C CNN
+F 3 "" H 5850 4300 60  0000 C CNN
+	1    5850 4300
+	1    0    0    -1
+$EndComp
+$Comp
+L +5V #PWR03
 U 1 1 55686CCD
-P 5950 2350
-F 0 "#PWR04" H 5950 2440 20  0001 C CNN
-F 1 "+5V" H 5950 2440 30  0000 C CNN
-F 2 "" H 5950 2350 60  0000 C CNN
-F 3 "" H 5950 2350 60  0000 C CNN
-	1    5950 2350
-	1    0    0    -1
-$EndComp
-Wire Wire Line
-	5950 2350 5950 3150
-Wire Wire Line
-	5950 2550 5350 2550
-Wire Wire Line
-	5350 2550 5350 2750
-Connection ~ 5950 2550
-Wire Wire Line
-	5650 2550 5650 2750
-Connection ~ 5650 2550
-$Comp
-L GND #PWR05
+P 5950 2300
+F 0 "#PWR03" H 5950 2390 20  0001 C CNN
+F 1 "+5V" H 5950 2390 30  0000 C CNN
+F 2 "" H 5950 2300 60  0000 C CNN
+F 3 "" H 5950 2300 60  0000 C CNN
+	1    5950 2300
+	1    0    0    -1
+$EndComp
+Wire Wire Line
+	5950 2300 5950 3100
+Wire Wire Line
+	5950 2500 5350 2500
+Wire Wire Line
+	5350 2500 5350 2700
+Connection ~ 5950 2500
+Wire Wire Line
+	5650 2500 5650 2700
+Connection ~ 5650 2500
+$Comp
+L GND #PWR04
 U 1 1 55686E81
-P 5350 4000
-F 0 "#PWR05" H 5350 4000 30  0001 C CNN
-F 1 "GND" H 5350 3930 30  0001 C CNN
-F 2 "" H 5350 4000 60  0000 C CNN
-F 3 "" H 5350 4000 60  0000 C CNN
-	1    5350 4000
-	1    0    0    -1
-$EndComp
-Wire Wire Line
-	5350 4000 5350 3150
-Wire Wire Line
-	5450 3850 5350 3850
-Connection ~ 5350 3850
-Wire Wire Line
-	5650 3150 5650 3250
-Wire Wire Line
-	5650 3250 5350 3250
-Connection ~ 5350 3250
+P 5350 3950
+F 0 "#PWR04" H 5350 3950 30  0001 C CNN
+F 1 "GND" H 5350 3880 30  0001 C CNN
+F 2 "" H 5350 3950 60  0000 C CNN
+F 3 "" H 5350 3950 60  0000 C CNN
+	1    5350 3950
+	1    0    0    -1
+$EndComp
+Wire Wire Line
+	5350 3950 5350 3100
+Wire Wire Line
+	5450 3800 5350 3800
+Connection ~ 5350 3800
+Wire Wire Line
+	5650 3100 5650 3200
+Wire Wire Line
+	5650 3200 5350 3200
+Connection ~ 5350 3200
 $Comp
 L CP1 C3
 U 1 1 55686FA6
-P 7350 5150
-F 0 "C3" H 7400 5250 50  0000 L CNN
-F 1 "CP1" H 7400 5050 50  0000 L CNN
-F 2 "~" H 7350 5150 60  0000 C CNN
-F 3 "~" H 7350 5150 60  0000 C CNN
-	1    7350 5150
-	1    0    0    -1
-$EndComp
-Wire Wire Line
-	7050 4750 7350 4750
-Wire Wire Line
-	7350 4750 7350 4950
-$Comp
-L GND #PWR06
+P 7350 5100
+F 0 "C3" H 7400 5200 50  0000 L CNN
+F 1 "CP1" H 7400 5000 50  0000 L CNN
+F 2 "~" H 7350 5100 60  0000 C CNN
+F 3 "~" H 7350 5100 60  0000 C CNN
+	1    7350 5100
+	1    0    0    -1
+$EndComp
+Wire Wire Line
+	7050 4700 7350 4700
+Wire Wire Line
+	7350 4700 7350 4900
+$Comp
+L GND #PWR05
 U 1 1 55686FDA
-P 7350 5550
-F 0 "#PWR06" H 7350 5550 30  0001 C CNN
-F 1 "GND" H 7350 5480 30  0001 C CNN
-F 2 "" H 7350 5550 60  0000 C CNN
-F 3 "" H 7350 5550 60  0000 C CNN
-	1    7350 5550
-	1    0    0    -1
-$EndComp
-Wire Wire Line
-	7350 5550 7350 5350
-Wire Wire Line
-	3800 3600 5000 3600
-Wire Wire Line
-	5000 3600 5000 4650
-Wire Wire Line
-	5000 4650 5450 4650
+P 7350 5500
+F 0 "#PWR05" H 7350 5500 30  0001 C CNN
+F 1 "GND" H 7350 5430 30  0001 C CNN
+F 2 "" H 7350 5500 60  0000 C CNN
+F 3 "" H 7350 5500 60  0000 C CNN
+	1    7350 5500
+	1    0    0    -1
+$EndComp
+Wire Wire Line
+	7350 5500 7350 5300
 NoConn ~ 3250 3100
 NoConn ~ 2950 3100
@@
 NoConn ~ 3800 5050
 NoConn ~ 3800 4950
-NoConn ~ 3800 4300
-NoConn ~ 3800 4200
-NoConn ~ 3800 4100
-NoConn ~ 3800 4000
-NoConn ~ 3800 3900
-NoConn ~ 7050 3550
+NoConn ~ 7050 3500
 NoConn ~ 2400 5550
 NoConn ~ 2400 5450
@@
 $EndComp
 Wire Wire Line
-	5450 4250 5150 4250
-Wire Wire Line
-	5150 4250 5150 3800
-Wire Wire Line
-	5150 3800 3800 3800
-Wire Wire Line
 	4200 2800 4200 2900
 Wire Wire Line
@@
 Wire Wire Line
 	4800 2800 4800 2900
-Wire Wire Line
-	4200 4550 4200 3300
-Wire Wire Line
-	4400 4650 4400 3300
-Wire Wire Line
-	4600 4750 4600 3300
-Wire Wire Line
-	4800 4850 4800 3300
-$Comp
-L +5V #PWR?
+$Comp
+L +5V #PWR06
 U 1 1 556894CB
 P 4500 2100
-F 0 "#PWR?" H 4500 2190 20  0001 C CNN
+F 0 "#PWR06" H 4500 2190 20  0001 C CNN
 F 1 "+5V" H 4500 2190 30  0000 C CNN
 F 2 "" H 4500 2100 60  0000 C CNN
@@
 	4600 2300 4600 2200
 Connection ~ 4600 2200
-$Comp
-L RESONATEUR Y?
-U 1 1 55689636
-P 7800 4150
-F 0 "Y?" H 7820 4350 60  0000 C CNN
-F 1 "RESONATEUR" H 8230 3950 60  0000 C CNN
-F 2 "" H 7800 4150 60  0000 C CNN
-F 3 "" H 7800 4150 60  0000 C CNN
-	1    7800 4150
+Wire Wire Line
+	7050 3900 7150 3900
+Wire Wire Line
+	7150 3900 7150 3800
+Wire Wire Line
+	7150 3800 7450 3800
+Wire Wire Line
+	7050 4300 7150 4300
+Wire Wire Line
+	7150 4300 7150 4400
+Wire Wire Line
+	7150 4400 7450 4400
+$Comp
+L GND #PWR07
+U 1 1 556AA04A
+P 7850 4350
+F 0 "#PWR07" H 7850 4350 30  0001 C CNN
+F 1 "GND" H 7850 4280 30  0001 C CNN
+F 2 "" H 7850 4350 60  0000 C CNN
+F 3 "" H 7850 4350 60  0000 C CNN
+	1    7850 4350
+	1    0    0    -1
+$EndComp
+Wire Wire Line
+	7850 4100 7850 4350
+Wire Wire Line
+	3800 4100 4400 4100
+Wire Wire Line
+	4400 4100 4400 3300
+Wire Wire Line
+	3800 4000 4200 4000
+Wire Wire Line
+	4200 4000 4200 3300
+NoConn ~ 3800 3900
+NoConn ~ 3800 4750
+NoConn ~ 3800 4850
+NoConn ~ 3800 3800
+NoConn ~ 3800 3600
+Wire Wire Line
+	3800 4550 4600 4550
+Wire Wire Line
+	4600 4550 4600 3300
+Wire Wire Line
+	3800 4650 4800 4650
+Wire Wire Line
+	4800 4650 4800 3300
+$Comp
+L CSTLS_G Q1
+U 1 1 556AA4EB
+P 7450 4100
+F 0 "Q1" H 7270 4230 50  0000 L BNN
+F 1 "CSTLS_G" H 7520 4230 50  0000 L BNN
+F 2 "murata-resonators-CSTLS_G8" H 7450 4250 50  0001 C CNN
+F 3 "" H 7450 4100 60  0000 C CNN
+	1    7450 4100
 	0    -1   -1   0
 $EndComp
 Wire Wire Line
-	7050 3950 7300 3950
-Wire Wire Line
-	7300 3950 7300 3850
-Wire Wire Line
-	7300 3850 7750 3850
-Wire Wire Line
-	7050 4350 7300 4350
-Wire Wire Line
-	7300 4350 7300 4450
-Wire Wire Line
-	7300 4450 7750 4450
+	7450 3800 7450 3900
+Wire Wire Line
+	7450 4400 7450 4300
+Wire Wire Line
+	7850 4100 7750 4100
+Wire Wire Line
+	3800 4300 5300 4300
+Wire Wire Line
+	5300 4300 5300 4200
+Wire Wire Line
+	5300 4200 5450 4200
+Wire Wire Line
+	3800 4200 5000 4200
+Wire Wire Line
+	5000 4200 5000 4600
+Wire Wire Line
+	5000 4600 5450 4600
 $EndSCHEMATC

Commit message: re-layed out with correct mouse part
Connections:
- wire segments 47 -> 49
Changed lines of the file:
@@
 NoConn ~ 2400 5550
 NoConn ~ 2400 5450
-NoConn ~ 3800 3700
 $Comp
 L ARDUINO_MINI U1
@@
 Wire Wire Line
 	7850 4100 7850 4350
-Wire Wire Line
-	3800 4100 4400 4100
-Wire Wire Line
-	4400 4100 4400 3300
-Wire Wire Line
-	3800 4000 4200 4000
-Wire Wire Line
-	4200 4000 4200 3300
-NoConn ~ 3800 3900
-NoConn ~ 3800 4750
-NoConn ~ 3800 4850
-NoConn ~ 3800 3800
 NoConn ~ 3800 3600
 Wire Wire Line
-	3800 4550 4600 4550
+	4600 3300 4600 4750
 Wire Wire Line
-	4600 4550 4600 3300
-Wire Wire Line
-	3800 4650 4800 4650
-Wire Wire Line
-	4800 4650 4800 3300
+	4800 3300 4800 4850
 $Comp
 L CSTLS_G Q1
@@
 	7850 4100 7750 4100
 Wire Wire Line
-	3800 4300 5300 4300
+	4500 4600 5450 4600
 Wire Wire Line
-	5300 4300 5300 4200
+	4800 4850 3800 4850
 Wire Wire Line
-	5300 4200 5450 4200
+	4600 4750 3800 4750
 Wire Wire Line
-	3800 4200 5000 4200
+	4500 4650 3800 4650
 Wire Wire Line
-	5000 4200 5000 4600
+	4500 4600 4500 4650
 Wire Wire Line
-	5000 4600 5450 4600
+	3800 4550 4400 4550
+Wire Wire Line
+	4400 4550 4400 4500
+Wire Wire Line
+	4400 4500 5350 4500
+Wire Wire Line
+	5350 4500 5350 4200
+Wire Wire Line
+	5350 4200 5450 4200
+NoConn ~ 3800 4200
+NoConn ~ 3800 4300
+Wire Wire Line
+	3800 3700 4200 3700
+Wire Wire Line
+	4200 3700 4200 3300
+Wire Wire Line
+	3800 3800 4400 3800
+Wire Wire Line
+	4400 3800 4400 3300
+NoConn ~ 3800 3900
+NoConn ~ 3800 4000
+NoConn ~ 3800 4100
 $EndSCHEMATC
