File: optical_mouse/optical_mouse.kicad_pcb (KiCad board)
At the start: 2 copper layers, 48.3 x 45.7 mm, 19 parts, among them Q1 CSTLS_G, U1 NANO

Commit message: tweak fill
Routing:
- net N-0000019: track 28.5 -> 27.0 mm
Other:
- board text added: "OptiMouseCam v1.0 (C) 2015 Dave Berkeley"
- board text removed: "OptMouseCam v1.0 (C) 2015 Dave Berkeley"
Changed lines of the file:
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@@
     (thickness 1.6)
     (drawings 5)
-    (tracks 90)
+    (tracks 92)
     (zones 0)
     (modules 19)
@@
     )
   )
-  (gr_text "OptMouseCam v1.0 (C) 2015 Dave Berkeley" (at 154.94 128.27 90) (layer B.SilkS)
+  (gr_text "OptiMouseCam v1.0 (C) 2015 Dave Berkeley" (at 154.94 128.27 90) (layer B.SilkS)
     (effects (font (size 0.8 0.8) (thickness 0.2)))
   )
@@
   (segment (start 171.45 133.35) (end 179.07 133.35) (width 0.254) (layer B.Cu) (net 4))
   (segment (start 162.56 135.89) (end 170.18 135.89) (width 0.254) (layer B.Cu) (net 5))
-  (segment (start 162.56 110.49) (end 163.83 110.49) (width 0.254) (layer B.Cu) (net 6))
+  (segment (start 162.56 110.49) (end 165.1 110.49) (width 0.254) (layer B.Cu) (net 6))
   (segment (start 175.26 118.11) (end 181.61 118.11) (width 0.254) (layer B.Cu) (net 6))
-  (segment (start 175.26 109.22) (end 175.26 118.11) (width 0.254) (layer B.Cu) (net 6))
-  (segment (start 165.1 109.22) (end 175.26 109.22) (width 0.254) (layer B.Cu) (net 6))
-  (segment (start 163.83 110.49) (end 165.1 109.22) (width 0.254) (layer B.Cu) (net 6))
+  (segment (start 175.26 111.76) (end 175.26 118.11) (width 0.254) (layer B.Cu) (net 6))
+  (segment (start 171.45 111.76) (end 175.26 111.76) (width 0.254) (layer B.Cu) (net 6))
+  (segment (start 168.91 109.22) (end 171.45 111.76) (width 0.254) (layer B.Cu) (net 6))
+  (segment (start 166.37 109.22) (end 168.91 109.22) (width 0.254) (layer B.Cu) (net 6))
+  (segment (start 165.1 110.49) (end 166.37 109.22) (width 0.254) (layer B.Cu) (net 6))
   (segment (start 162.56 130.81) (end 170.62958 130.81) (width 0.254) (layer B.Cu) (net 7))
   (segment (start 170.62958 130.81) (end 171.02074 130.41884) (width 0.254) (layer B.Cu) (net 7))
